Commit message: my_robot v1 with colors

File: src/my_robot/urdf/my_robot.xacro (robot description, xacro)
@@ -1,4 +1,5 @@
 <?xml version="1.0"?>
 <robot name="my_robot" xmlns:xacro="http://www.ros.org/wiki/xacro">
+    <xacro:include filename="$(find my_robot)/urdf/my_robot.gazebo"/>
     <link name="robot_footprint"></link>
     <joint name="robot_footprint_joint" type="fixed">
@@ -60,5 +61,5 @@
         <inertial>
             <mass value="5"/>
-            <origin xyz="0 0 0" rpy=" 0 0 0"/>
+            <origin xyz="0 0 0" rpy=" 0 1.5707 1.5707"/>
             <inertia
                 ixx="0.1" ixy="0" ixz="0"
@@ -73,29 +74,5 @@
             </geometry>
         </collision>
-        <visual name="visual">
-            <origin xyz="0 0 0" rpy=" 0 1.5707 1.5707"/>
-            <geometry>
-                <cylinder radius=".1" length=".05"/>
-            </geometry>
-        </visual>
-    </link>
-    <!-- Right Wheel -->
-    <link name="right_wheel">
-        <inertial>
-            <mass value="5"/>
-            <origin xyz="0 0 0" rpy=" 0 0 0"/>
-            <inertia
-                ixx="0.1" ixy="0" ixz="0"
-                iyy="0.1" iyz="0"
-                izz="0.1"
-            />
-        </inertial>
-        <collision name="collision">
-            <origin xyz="0 0 0" rpy=" 0 1.5707 1.5707"/>
-            <geometry>
-                <cylinder radius=".1" length=".05"/>
-            </geometry>
-        </collision>
-        <visual name="visual">
+        <visual name="left_wheel_visual">
             <origin xyz="0 0 0" rpy=" 0 1.5707 1.5707"/>
             <geometry>
@@ -112,4 +89,28 @@
         <dynamics damping="1.0" friction="1.0"/>
     </joint>
+    <!-- Right Wheel -->
+    <link name="right_wheel">
+        <inertial>
+            <mass value="5"/>
+            <origin xyz="0 0 0" rpy=" 0 1.5707 1.5707"/>
+            <inertia
+                ixx="0.1" ixy="0" ixz="0"
+                iyy="0.1" iyz="0"
+                izz="0.1"
+            />
+        </inertial>
+        <collision name="collision">
+            <origin xyz="0 0 0" rpy=" 0 1.5707 1.5707"/>
+            <geometry>
+                <cylinder radius=".1" length=".05"/>
+            </geometry>
+        </collision>
+        <visual name="right_wheel_visual">
+            <origin xyz="0 0 0" rpy=" 0 1.5707 1.5707"/>
+            <geometry>
+                <cylinder radius=".1" length=".05"/>
+            </geometry>
+        </visual>
+    </link>
     <joint type="continuous" name="right_wheel_hinge">
         <origin xyz="0 -0.15 0" rpy="0 0 0"/>
@@ -124,5 +125,5 @@
         <inertial>
             <mass value="0.1"/>
-            <origin xyz="0 0 0" rpy=" 0 0 0"/>
+            <origin xyz="0.0 0 0" rpy=" 0 0 0"/>
             <inertia
                 ixx="1e-6" ixy="0" ixz="0"
@@ -131,19 +132,19 @@
             />
         </inertial>
-        <collision name="collision">
-            <origin xyz="0 0 0" rpy=" 0 0 0"/>
+        <collision name="camera_collision">
+            <origin xyz="0.0 0 0" rpy=" 0 0 0"/>
             <geometry>
-                <box size=".05 .05 .05"/>
+                <box size="0.05 0.05 0.05"/>
             </geometry>
         </collision>
-        <visual name="visual">
-            <origin xyz="0 0 0" rpy=" 0 0 0"/>
+        <visual name="camera_visual">
+            <origin xyz="0.0 0 0" rpy=" 0 0 0"/>
             <geometry>
-                <box size=".05 .05 .05"/>
+                <box size="0.05 0.05 0.05"/>
             </geometry>
         </visual>
     </link>
     <joint name="camera_joint" type="fixed">
-        <orgin xyz="0.2 0 0" rpy="0 0 0"/>
+        <origin xyz="0.2 0 0" rpy="0 0 0"/>
         <child link="camera"/>
         <parent link="chassis"/>
@@ -154,5 +155,5 @@
         <inertial>
             <mass value="1e-5"/>
-            <origin xyz="0 0 0" rpy=" 0 0 0"/>
+            <origin xyz="0.0 0 0" rpy=" 0 0 0"/>
             <inertia
                 ixx="1e-6" ixy="0" ixz="0"
@@ -161,16 +162,22 @@
             />
         </inertial>
-        <collision name="collision">
-            <origin xyz="0 0 0" rpy=" 0 0 0"/>
+        <collision name="hokuyo_collision">
+            <origin xyz="0.0 0 0" rpy=" 0 0 0"/>
             <geometry>
-                <box size=".01 .01 .01"/>
+                <box size="0.1 0.1 0.1"/>
             </geometry>
         </collision>
-        <visual name="visual">
-            <origin xyz="0 0 0" rpy=" 0 0 0"/>
+        <visual name="hokuyo_visual">
+            <origin xyz="0.0 0 0" rpy=" 0 0 0"/>
             <geometry>
-                <uri >package://</uri>
+                <mesh filename="package://my_robot/meshes/hokuyo.dae"/>
             </geometry>
         </visual>
     </link>
+    <joint name="hokuyo_joint" type="fixed">
+        <origin xyz="0.15 0 0.1" rpy="0 0 0"/>
+        <child link="hokuyo"/>
+        <parent link="chassis"/>
+        <axis xyz="0 1 0" rpy="0 0 0"/>
+    </joint>
 </robot>
